File: pcb/U3A_rs232.kicad_sch (KiCad schematic)
At the start: 16 parts, among them J1 Conn_02x05_Odd_Even, J2 Conn_01x07_Socket, J4 Conn_01x08_Socket, U1 MAX3232

Commit message: Adapt partlist vendors
Parts:
- H1, H2: Vendor HTL -> HTL, DigiKey; VendorId 101176 -> 100991, 100993, 732-12987-ND
Changed lines of the file:
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@@
       (effects (font (size 1.27 1.27)) hide)
     )
-    (property "Vendor" "HTL" (at 215.9 151.13 0)
-      (effects (font (size 1.27 1.27)) hide)
-    )
-    (property "VendorId" "101176" (at 215.9 151.13 0)
+    (property "Vendor" "HTL, DigiKey" (at 215.9 151.13 0)
+      (effects (font (size 1.27 1.27)) hide)
+    )
+    (property "VendorId" "100991, 100993, 732-12987-ND" (at 215.9 151.13 0)
       (effects (font (size 1.27 1.27)) hide)
     )
@@
       (effects (font (size 1.27 1.27)) hide)
     )
-    (property "Vendor" "HTL" (at 205.74 151.13 0)
-      (effects (font (size 1.27 1.27)) hide)
-    )
-    (property "VendorId" "101176" (at 205.74 151.13 0)
-      (effects (font (size 1.27 1.27)) hide)
-    )
+    (property "Vendor" "HTL, DigiKey" (at 205.74 151.13 0)
+      (effects (font (size 1.27 1.27)) hide)
+    )
+    (property "VendorId" "100991, 100993, 732-12987-ND" (at 205.74 151.13 0)
+      (effects (font (size 1.27 1.27)) hide)
+    )

Commit message: Update to KiCAD 9
Parts:
- FID1, FID2, FID3, FID4, H1, H2: now left out of the parts list

Commit message: Rename/Add/Remove bom fields
Parts:
- C1: HTL (none) -> 100140; Vendor HTL -> (none); VendorId 100140 -> (none)
- C2, C3: HTL (none) -> 100128; Vendor HTL -> (none); VendorId 100128 -> (none)
- C4, C5, C6: HTL (none) -> 103260; Vendor HTL -> (none); VendorId 103260 -> (none)
- H1, H2: DigiKey (none) -> 732-12987-ND; HTL (none) -> 100991, 100993; Vendor HTL, DigiKey -> (none); VendorId 100991, 100993, 732-12987-ND -> (none)
- J1: HTL (none) -> 101532; Vendor HTL -> (none); VendorId 101532 -> (none)
- J2, J4: HTL (none) -> 101546; Vendor HTL -> (none); VendorId 101546 -> (none)
- U1: HTL (none) -> 100294; Vendor HTL -> (none); VendorId 100294 -> (none)
Changed lines of the file:
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@@
 			)
 		)
-		(property "Vendor" "HTL, DigiKey"
-			(at 215.9 151.13 0)
-			(effects
-				(font
-					(size 1.27 1.27)
-				)
-				(hide yes)
-			)
-		)
-		(property "VendorId" "100991, 100993, 732-12987-ND"
-			(at 215.9 151.13 0)
+		(property "HTL" "100991, 100993"
+			(at 215.9 151.13 90)
+			(effects
+				(font
+					(size 1.27 1.27)
+				)
+				(hide yes)
+			)
+		)
+		(property "DigiKey" "732-12987-ND"
+			(at 215.9 151.13 90)
 			(effects
 				(font
@@
 			)
 		)
-		(property "Vendor" ""
-			(at 254 152.4 0)
-			(effects
-				(font
-					(size 1.27 1.27)
-				)
-				(hide yes)
-			)
-		)
-		(property "VendorId" ""
-			(at 254 152.4 0)
+		(property "DigiKey" ""
+			(at 254 152.4 90)
 			(effects
 				(font
@@
 			)
 		)
-		(property "Vendor" "HTL"
-			(at 166.37 66.04 0)
-			(effects
-				(font
-					(size 1.27 1.27)
-				)
-				(hide yes)
-			)
-		)
-		(property "VendorId" "103260"
-			(at 166.37 66.04 0)
+		(property "HTL" "103260"
+			(at 166.37 66.04 90)
+			(effects
+				(font
+					(size 1.27 1.27)
+				)
+				(hide yes)
+			)
+		)
+		(property "DigiKey" ""
+			(at 166.37 66.04 90)
 			(effects
 				(font
@@
 			)
 		)
-		(property "Vendor" ""
-			(at 228.6 152.4 0)
-			(effects
-				(font
-					(size 1.27 1.27)
-				)
-				(hide yes)
-			)
-		)
-		(property "VendorId" ""
-			(at 228.6 152.4 0)
+		(property "DigiKey" ""
+			(at 228.6 152.4 90)
 			(effects
 				(font
@@
 			)
 		)
-		(property "Vendor" ""
-			(at 266.7 152.4 0)
-			(effects
-				(font
-					(size 1.27 1.27)
-				)
-				(hide yes)
-			)
-		)
-		(property "VendorId" ""
-			(at 266.7 152.4 0)
+		(property "DigiKey" ""
+			(at 266.7 152.4 90)
 			(effects
 				(font
@@
 			)
 		)
-		(property "Vendor" "HTL"
+		(property "HTL" "100140"
 			(at 101.6 177.8 0)
 			(effects
@@
 			)
 		)
-		(property "VendorId" "100140"
+		(property "DigiKey" ""
 			(at 101.6 177.8 0)
 			(effects
@@
 			)
 		)
-		(property "Vendor" ""
-			(at 241.3 152.4 0)
-			(effects
-				(font
-					(size 1.27 1.27)
-				)
-				(hide yes)
-			)
-		)
-		(property "VendorId" ""
-			(at 241.3 152.4 0)
+		(property "DigiKey" ""
+			(at 241.3 152.4 90)
 			(effects
 				(font
@@
 			)
 		)
-		(property "Vendor" "HTL, DigiKey"
-			(at 205.74 151.13 0)
-			(effects
-				(font
-					(size 1.27 1.27)
-				)
-				(hide yes)
-			)
-		)
-		(property "VendorId" "100991, 100993, 732-12987-ND"
-			(at 205.74 151.13 0)
+		(property "HTL" "100991, 100993"
+			(at 205.74 151.13 90)
+			(effects
+				(font
+					(size 1.27 1.27)
+				)
+				(hide yes)
+			)
+		)
+		(property "DigiKey" "732-12987-ND"
+			(at 205.74 151.13 90)
 			(effects
 				(font
@@
 			)
 		)
-		(property "Vendor" "HTL"
+		(property "HTL" "101532"
 			(at 195.58 71.12 0)
 			(effects
@@
 			)
 		)
-		(property "VendorId" "101532"
+		(property "DigiKey" ""
 			(at 195.58 71.12 0)
 			(effects
@@
 			)
 		)
-		(property "Vendor" "HTL"
+		(property "HTL" "100128"
 			(at 116.84 57.15 0)
 			(effects
@@
 			)
 		)
-		(property "VendorId" "100128"
+		(property "DigiKey" ""
 			(at 116.84 57.15 0)
 			(effects
@@
 			)
 		)
-		(property "Vendor" "HTL"
+		(property "HTL" "100128"
 			(at 114.3 177.8 0)
 			(effects
@@
 			)
 		)
-		(property "VendorId" "100128"
+		(property "DigiKey" ""
 			(at 114.3 177.8 0)
 			(effects
@@
 			)
 		)
-		(property "Vendor" "HTL"
+		(property "HTL" "103260"
 			(at 162.56 57.15 0)
 			(effects
@@
 			)
 		)
-		(property "VendorId" "103260"
+		(property "DigiKey" ""
 			(at 162.56 57.15 0)
 			(effects
@@
 			)
 		)
-		(property "Vendor" "HTL"
+		(property "HTL" "100294"
 			(at 139.7 76.2 0)
 			(effects
@@
 			)
 		)
-		(property "VendorId" "100294"
+		(property "DigiKey" ""
 			(at 139.7 76.2 0)
 			(effects
@@
 			)
 		)
-		(property "Vendor" "HTL"
-			(at 109.22 144.78 0)
-			(effects
-				(font
-					(size 1.27 1.27)
-				)
-				(hide yes)
-			)
-		)
-		(property "VendorId" "101546"
-			(at 109.22 144.78 0)
+		(property "HTL" "101546"
+			(at 109.22 144.78 90)
+			(effects
+				(font
+					(size 1.27 1.27)
+				)
+				(hide yes)
+			)
+		)
+		(property "DigiKey" ""
+			(at 109.22 144.78 90)
 			(effects
 				(font
@@
 			)
 		)
-		(property "Vendor" "HTL"
-			(at 99.06 90.17 0)
-			(effects
-				(font
-					(size 1.27 1.27)
-				)
-				(hide yes)
-			)
-		)
-		(property "VendorId" "101546"
-			(at 99.06 90.17 0)
+		(property "HTL" "101546"
+			(at 99.06 90.17 90)
+			(effects
+				(font
+					(size 1.27 1.27)
+				)
+				(hide yes)
+			)
+		)
+		(property "DigiKey" ""
+			(at 99.06 90.17 90)
 			(effects
 				(font
@@
 			)
 		)
-		(property "Vendor" "HTL"
-			(at 166.37 73.66 0)
-			(effects
-				(font
-					(size 1.27 1.27)
-				)
-				(hide yes)
-			)
-		)
-		(property "VendorId" "103260"
-			(at 166.37 73.66 0)
-			(effects
-				(font
+		(property "HTL" "103260"
+			(at 166.37 73.66 90)
+			(effects
+				(font
+					(size 1.27 1.27)
+				)
+				(hide yes)
+			)
+		)
+		(property "DigiKey" ""
+			(at 166.37 73.66 90)
+			(effects
+				(font
